Commit message: Tmp: tyring to build multi sima simulation but failed. Send commit and is going to start a new branch from previous commit to try simulation by using domain bridge.
Note: This isn't finish yet, some nodes and topic isn't push to the right namespace yet. Can use rqt_graph to check out. Maybe is the vl53 bridge that haven't push to the right namespace. By the way, the namespace need more adjustment since it's complicated and not clearly and bad now.

File: SIMA-ws/src/gazebo_sim_bot/urdf/my_robot.urdf.xacro (robot description, xacro)
@@ -1,4 +1,6 @@
 <?xml version="1.0"?>
 <robot name="sima_robot" xmlns:xacro="http://www.ros.org/wiki/xacro">
+  <xacro:arg name="robot_name" default=""/>
+  <xacro:property name="prefix" value="$(arg robot_name)"/>
   <material name="blue">
     <color rgba="0 0 0.8 1"/>
@@ -13,11 +15,11 @@
     <color rgba="1 0 0 1"/>
   </material>
-  <link name="base_footprint"/>
-  <joint name="base_joint" type="fixed">
-    <parent link="base_footprint"/>
-    <child link="base_link"/>
+  <link name="${prefix}base_footprint"/>
+  <joint name="${prefix}base_joint" type="fixed">
+    <parent link="${prefix}base_footprint"/>
+    <child link="${prefix}base_link"/>
     <origin xyz="0 0 0.105" rpy="0 0 0"/>
   </joint>
-  <link name="base_link">
+  <link name="${prefix}base_link">
     <visual>
       <geometry>
@@ -36,5 +38,5 @@
     </inertial>
   </link>
-  <link name="left_wheel">
+  <link name="${prefix}left_wheel">
     <visual>
       <geometry>
@@ -53,11 +55,11 @@
     </inertial>
   </link>
-  <joint name="left_wheel_joint" type="continuous">
-    <parent link="base_link"/>
-    <child link="left_wheel"/>
+  <joint name="${prefix}left_wheel_joint" type="continuous">
+    <parent link="${prefix}base_link"/>
+    <child link="${prefix}left_wheel"/>
     <origin xyz="0 0.085 -0.075" rpy="-1.57 0 0"/>
     <axis xyz="0 0 1"/>
   </joint>
-  <link name="right_wheel">
+  <link name="${prefix}right_wheel">
     <visual>
       <geometry>
@@ -76,11 +78,11 @@
     </inertial>
   </link>
-  <joint name="right_wheel_joint" type="continuous">
-    <parent link="base_link"/>
-    <child link="right_wheel"/>
+  <joint name="${prefix}right_wheel_joint" type="continuous">
+    <parent link="${prefix}base_link"/>
+    <child link="${prefix}right_wheel"/>
     <origin xyz="0 -0.085 -0.075" rpy="-1.57 0 0"/>
     <axis xyz="0 0 1"/>
   </joint>
-  <link name="front_caster">
+  <link name="${prefix}front_caster">
     <visual>
       <geometry>
@@ -99,10 +101,10 @@
     </inertial>
   </link>
-  <joint name="front_caster_joint" type="fixed">
-    <parent link="base_link"/>
-    <child link="front_caster"/>
+  <joint name="${prefix}front_caster_joint" type="fixed">
+    <parent link="${prefix}base_link"/>
+    <child link="${prefix}front_caster"/>
     <origin xyz="0.06 0 -0.09"/>
   </joint>
-  <link name="back_caster">
+  <link name="${prefix}back_caster">
     <visual>
       <geometry>
@@ -121,10 +123,10 @@
     </inertial>
   </link>
-  <joint name="back_caster_joint" type="fixed">
-    <parent link="base_link"/>
-    <child link="back_caster"/>
+  <joint name="${prefix}back_caster_joint" type="fixed">
+    <parent link="${prefix}base_link"/>
+    <child link="${prefix}back_caster"/>
     <origin xyz="-0.06 0 -0.09"/>
   </joint>
-  <gazebo reference="left_wheel">
+  <gazebo reference="${prefix}left_wheel">
     <mu1>10.0</mu1>
     <mu2>10.0</mu2>
@@ -135,5 +137,5 @@
     <material>Gazebo/White</material>
   </gazebo>
-  <gazebo reference="right_wheel">
+  <gazebo reference="${prefix}right_wheel">
     <mu1>10.0</mu1>
     <mu2>10.0</mu2>
@@ -144,5 +146,5 @@
     <material>Gazebo/White</material>
   </gazebo>
-  <gazebo reference="front_caster">
+  <gazebo reference="${prefix}front_caster">
     <mu1>0.001</mu1>
     <mu2>0.001</mu2>
@@ -153,5 +155,5 @@
     <material>Gazebo/Black</material>
   </gazebo>
-  <gazebo reference="back_caster">
+  <gazebo reference="${prefix}back_caster">
     <mu1>0.001</mu1>
     <mu2>0.001</mu2>
@@ -163,5 +165,5 @@
   </gazebo>
   <xacro:macro name="vl53_sensor" params="name x y yaw color topic_name">
-    <link name="${name}_link">
+    <link name="${prefix}${name}_link">
       <visual>
         <geometry>
@@ -180,11 +182,11 @@
       </inertial>
     </link>
-    <joint name="${name}_joint" type="fixed">
-      <parent link="base_link"/>
-      <child link="${name}_link"/>
+    <joint name="${prefix}${name}_joint" type="fixed">
+      <parent link="${prefix}base_link"/>
+      <child link="${prefix}${name}_link"/>
       <origin xyz="${x} ${y} 0.0" rpy="0 0 ${yaw}"/>
     </joint>
-    <gazebo reference="${name}_link">
-      <sensor name="${name}" type="ray">
+    <gazebo reference="${prefix}${name}_link">
+      <sensor name="${prefix}${name}" type="ray">
         <pose>0 0 0 0 0 0</pose>
         <always_on>true</always_on>
@@ -205,11 +207,11 @@
             <stddev>0.01</stddev> </noise>
         </ray>
-        <plugin name="${name}_controller" filename="libgazebo_ros_ray_sensor.so">
+        <plugin name="${prefix}${name}_controller" filename="libgazebo_ros_ray_sensor.so">
             <ros>
-                <namespace>/</namespace>
+                <namespace>${prefix}</namespace>
                 <remapping>~/out:=${topic_name}</remapping>
             </ros>
             <output_type>sensor_msgs/LaserScan</output_type>
-            <frame_name>${name}_link</frame_name>
+            <frame_name>${prefix}${name}_link</frame_name>
             <radiation_type>infrared</radiation_type>
         </plugin>
@@ -217,14 +219,14 @@
     </gazebo>
   </xacro:macro>
-    <xacro:vl53_sensor name="sensor_left"   x="0.075" y="0.075"  yaw="0.785"  color="red" topic_name="/sim/vl53_left"/>
-    <xacro:vl53_sensor name="sensor_center" x="0.08"  y="0.0"    yaw="0.0"    color="red" topic_name="/sim/vl53_center"/>
-    <xacro:vl53_sensor name="sensor_right"  x="0.075" y="-0.075" yaw="-0.785" color="red" topic_name="/sim/vl53_right"/>
+    <xacro:vl53_sensor name="sensor_left"   x="0.075" y="0.075"  yaw="0.785"  color="red" topic_name="sim/vl53_left"/>
+    <xacro:vl53_sensor name="sensor_center" x="0.08"  y="0.0"    yaw="0.0"    color="red" topic_name="sim/vl53_center"/>
+    <xacro:vl53_sensor name="sensor_right"  x="0.075" y="-0.075" yaw="-0.785" color="red" topic_name="sim/vl53_right"/>
   <gazebo>
     <plugin name="diff_drive" filename="libgazebo_ros_diff_drive.so">
       <ros>
-        <namespace></namespace>
+        <!-- DO NOT set namespace here - it's handled by PushRosNamespace in launch file -->
       </ros>
-      <left_joint>left_wheel_joint</left_joint>
-      <right_joint>right_wheel_joint</right_joint>
+      <left_joint>${prefix}left_wheel_joint</left_joint>
+      <right_joint>${prefix}right_wheel_joint</right_joint>
       <wheel_separation>0.17</wheel_separation>
       <wheel_diameter>0.06</wheel_diameter>
@@ -232,6 +234,6 @@
       <publish_odom_tf>true</publish_odom_tf>
       <publish_wheel_tf>true</publish_wheel_tf>
-      <odometry_frame>odom</odometry_frame>
-      <robot_base_frame>base_footprint</robot_base_frame>
+      <odometry_frame>${prefix}odom</odometry_frame>
+      <robot_base_frame>${prefix}base_footprint</robot_base_frame>
       <command_topic>cmd_vel</command_topic>
       <max_wheel_torque>20</max_wheel_torque>

Commit message: Add: Include ros2 domain bridge in dockerfile inorder to use domain bridge to accomplish multi robot simulation of navigation in gazebo. Now can run gazebo simulation in domain 1 and spawn 2 sima robot. Then can control (or navigate) two sima in domain 2 and domain 3 in different terminal respectively. Also, each sima can decide which watpoints (path and goal) it should go depends on it's location.
Detail changes:
- Modify docker-compose.yaml and Dockerfile to build the environment. (If image is already built, remember delete the image and rebuild to install necessary packages and tools)
- Add bridge_config.yaml to create domain bridge. (Will be included or created in sim.launch.py launch file in gazebo_sim_bot) (Here can decide which domain is used to control which sima in gazebo simulator)
- Add sim_vl53_publisher to publish simulated sensors' ranges data under different prefix. For example, /sima1/sensors/raw_ranges. (It will be remap to /sensors/raw_ranges by domain bridge to different domains, see bridge_config.yaml for more details)
- Fix robot urdf file to support multi robot. (Including spawning, publishing transforms, publishing sensors' simulated data)
- Change sim.launch.py to spawn multi sima. (The gazebo_sim_bot is launch by this file)
- Add tf_republisher.cpp in navigation2_run to republish /tf and /tf_static in correct frame id in nav2. (Otherwise needs to change lots of frame id names in code and it's stupid)
- Change sima_navigator.cpp to support dynamic path selecting depending on each robot's start position. Can change start points and waypoints in nav2_params_sima.yaml
- Modified nav2_params_sima.yaml, sim_launch.py to support the new features.

How to use (Total needs 4 terminal to simulate):
- To change domain id, for example you want to change to domain 1, run "export ROS_DOMAIN_ID=1"
- Run "ros2 launch gazebo_sim_bot sim.launch.py" in domain 1.
- Run "ros2 launch navigation2_run sim_launch.py remove_prefix:=sima1/" in domain 2.
- Run "ros2 launch navigation2_run sim_launch.py remove_prefix:=sima2/" in domain 3.
- Run "ros2 topic pub /start_sima std_msgs/msg/Bool {"data: true"}" in domain 1.

File: SIMA-ws/src/gazebo_sim_bot/urdf/my_robot.urdf.xacro (robot description, xacro)
@@ -13,5 +13,10 @@
     <color rgba="1 0 0 1"/>
   </material>
-  <link name="base_footprint"/>
+  <link name="base_footprint">
+    <inertial>
+      <mass value="0.0001"/>
+      <inertia ixx="0.000001" ixy="0.0" ixz="0.0" iyy="0.000001" iyz="0.0" izz="0.000001"/>
+    </inertial>
+  </link>
   <joint name="base_joint" type="fixed">
     <parent link="base_footprint"/>
@@ -162,5 +167,6 @@
     <material>Gazebo/Black</material>
   </gazebo>
-  <xacro:macro name="vl53_sensor" params="name x y yaw color topic_name">
+  <xacro:arg name="robot_name" default="sima1"/>
+  <xacro:macro name="vl53_sensor" params="name x y yaw color">
     <link name="${name}_link">
       <visual>
@@ -207,6 +213,6 @@
         <plugin name="${name}_controller" filename="libgazebo_ros_ray_sensor.so">
             <ros>
-                <namespace>/</namespace>
-                <remapping>~/out:=${topic_name}</remapping>
+                <namespace>/$(arg robot_name)</namespace>
+                <remapping>~/out:=${name}</remapping>
             </ros>
             <output_type>sensor_msgs/LaserScan</output_type>
@@ -217,11 +223,13 @@
     </gazebo>
   </xacro:macro>
-    <xacro:vl53_sensor name="sensor_left"   x="0.075" y="0.075"  yaw="0.785"  color="red" topic_name="/sim/vl53_left"/>
-    <xacro:vl53_sensor name="sensor_center" x="0.08"  y="0.0"    yaw="0.0"    color="red" topic_name="/sim/vl53_center"/>
-    <xacro:vl53_sensor name="sensor_right"  x="0.075" y="-0.075" yaw="-0.785" color="red" topic_name="/sim/vl53_right"/>
+    <xacro:vl53_sensor name="vl53_left"   x="0.075" y="0.075"  yaw="0.785"  color="red"/>
+    <xacro:vl53_sensor name="vl53_center" x="0.08"  y="0.0"    yaw="0.0"    color="red"/>
+    <xacro:vl53_sensor name="vl53_right"  x="0.075" y="-0.075" yaw="-0.785" color="red"/>
   <gazebo>
     <plugin name="diff_drive" filename="libgazebo_ros_diff_drive.so">
       <ros>
-        <namespace></namespace>
+        <namespace>/$(arg robot_name)</namespace>
+        <remapping>cmd_vel:=cmd_vel</remapping>
+        <remapping>odom:=odom</remapping>
       </ros>
       <left_joint>left_wheel_joint</left_joint>
@@ -230,12 +238,24 @@
       <wheel_diameter>0.06</wheel_diameter>
       <publish_odom>true</publish_odom>
-      <publish_odom_tf>true</publish_odom_tf>
-      <publish_wheel_tf>true</publish_wheel_tf>
+      <publish_odom_tf>false</publish_odom_tf>
+      <publish_wheel_tf>false</publish_wheel_tf>
+      <publish_wheel_joint_state>true</publish_wheel_joint_state>
       <odometry_frame>odom</odometry_frame>
       <robot_base_frame>base_footprint</robot_base_frame>
-      <command_topic>cmd_vel</command_topic>
       <max_wheel_torque>20</max_wheel_torque>
       <max_wheel_acceleration>2.0</max_wheel_acceleration>
     </plugin>
   </gazebo>
+  <gazebo>
+    <plugin name="gazebo_ros_p3d" filename="libgazebo_ros_p3d.so">
+      <ros>
+        <namespace>/$(arg robot_name)</namespace>
+        <remapping>odom:=ground_truth_pose</remapping>
+      </ros>
+      <frame_name>map</frame_name> <body_name>base_footprint</body_name> <update_rate>50.0</update_rate>
+      <xyz_offset>0 0 0</xyz_offset>
+      <rpy_offset>0 0 0</rpy_offset>
+      <gaussian_noise>0.0</gaussian_noise>
+    </plugin>
+  </gazebo>
 </robot>
